Commit message: Fix toddlerbot_3_0_2xc left arm: mirror from right (CAD config bug)
The shared arm CAD's `left_arm` config has a ~90° spurious shoulder_roll at
joint-zero, so the left arm exported sticking straight out instead of hanging.
Since the arm CAD is the original author's shared doc, fix at the model level:
rebuild the left arm as a Y-mirror of the (correct) right arm.

- scripts/mirror_left_arm.py: mirrors body/geom/inertial poses + joint axes,
  adds Y-mirrored mesh copies (assets/lmir_*.stl), across all 6 robot variants.
- Home keyframe arm joints set to 0 (arms hang vertically at zero after fix).
- Removed 10 orphaned old left-arm visual meshes; regenerated URDF.
- Verified: zero-pose & home Y-mirror symmetric, articulation mirrors correctly,
  mass unchanged (3.4522 kg), physics stable, all 6 variants load.
- BUILD.md updated with the fix + mcc reference.

Co-Authored-By: Claude Opus 4.8 <noreply@anthropic.com>

File: toddlerbot/descriptions/toddlerbot_3_0_2xc/toddlerbot_3_0_2xc.urdf (robot description, URDF)
Before this commit: robot toddlerbot_3_0_2xc, 91 links, 90 joints
Links:
- link left_elbow_gear_drive: geometry visual mesh filename=assets/lmir_right_elbow_gear_drive_visual.stl scale=1.0 1.0 1.0
- link left_elbow_roll_link: geometry collision box size=0.0409073 0.0582348 0.0576582 type=box; visual mesh filename=assets/lmir_right_elbow_roll_link_visual.stl scale=1.0 1.0 1.0
- link left_elbow_yaw_link: geometry collision box size=0.025985 0.0593 0.055126 type=box; visual mesh filename=assets/lmir_right_elbow_yaw_link_visual.stl scale=1.0 1.0 1.0
- link left_hand: geometry collision box size=0.074 0.05 0.02 type=box; visual mesh filename=assets/lmir_right_hand_visual.stl scale=1.0 1.0 1.0
- link left_shoulder_gear_drive: geometry visual mesh filename=assets/lmir_right_shoulder_gear_drive_visual.stl scale=1.0 1.0 1.0
- link left_shoulder_pitch_link: geometry visual mesh filename=assets/lmir_right_shoulder_pitch_link_visual.stl scale=1.0 1.0 1.0
- link left_shoulder_roll_link: geometry collision box size=0.0409073 0.0582348 0.0576582 type=box; visual mesh filename=assets/lmir_right_shoulder_roll_link_visual.stl scale=1.0 1.0 1.0
- link left_shoulder_yaw_link: geometry collision box size=0.046 0.025985 0.054214 type=box; visual mesh filename=assets/lmir_right_shoulder_yaw_link_visual.stl scale=1.0 1.0 1.0
- link left_wrist_gear_drive: geometry visual mesh filename=assets/lmir_right_wrist_gear_drive_visual.stl scale=1.0 1.0 1.0
- link left_wrist_pitch_link: geometry collision box size=0.0409073 0.0585832 0.0583139 type=box; visual mesh filename=assets/lmir_right_wrist_pitch_link_visual.stl scale=1.0 1.0 1.0
Joints:
- joint left_elbow_roll: origin xyz=-0.019 0.061 0.0 rpy=0.0 0.0 0.0 -> xyz=0.019 -0.0232927 -0.0563777 rpy=0.0 0.0 0.0
- joint left_elbow_yaw_drive: origin xyz=0.019 0.019 0.024 rpy=0.0 0.0 0.0 -> xyz=-0.019 0.0149263 -0.0267246 rpy=0.0 0.0 0.0
- joint left_elbow_yaw_driven: axis 0.0 1.0 0.0 -> 0.0 0.38176 0.924261; origin xyz=0.019 0.025 0.0 rpy=0.0 0.0 0.0 -> xyz=-0.019 -0.00954621 -0.0231056 rpy=0.0 0.0 0.0
- joint left_shoulder_pitch: axis 0.0 1.0 0.0 -> 0.0 -1.0 0.0; limit lower=-4.712388980384688 upper=4.7123889803846915 effort=100 velocity=100 -> lower=-4.71238898038469 upper=4.71238898038469 effort=100 velocity=100
- joint left_shoulder_roll: origin xyz=-0.019 0.027 -0.0107595 rpy=0.0 0.0 0.0 -> xyz=0.019 0.027 -0.0107595 rpy=0.0 0.0 0.0
- joint left_shoulder_yaw_drive: origin xyz=0.019 0.019 0.024 rpy=0.0 0.0 0.0 -> xyz=-0.019 0.0149263 -0.0267246 rpy=0.0 0.0 0.0
- joint left_shoulder_yaw_driven: axis 0.0 1.0 0.0 -> 0.0 0.38176 0.924261; origin xyz=0.019 0.025 0.0 rpy=0.0 0.0 0.0 -> xyz=-0.019 -0.00954621 -0.0231056 rpy=0.0 0.0 0.0
- joint left_wrist_pitch_drive: origin xyz=0.0 -0.024 -0.003 rpy=0.0 0.0 0.0 -> xyz=0.0 0.00639168 0.023327 rpy=0.0 0.0 0.0
- joint left_wrist_pitch_driven: axis 0.0 0.0 -1.0 -> 0.0 0.924261 -0.38176; origin xyz=0.0 0.061 0.022 rpy=0.0 0.0 0.0 -> xyz=0.0 -0.00295979 -0.0647784 rpy=0.0 0.0 0.0
- joint left_wrist_roll: origin xyz=-0.019 0.0 -0.022 rpy=0.0 0.0 0.0 -> xyz=0.019 -0.020333 0.00840066 rpy=0.0 0.0 0.0

Commit message: Fix toddlerbot_3_0_2xc right leg: mirror from left (CAD config bug)
Same class of bug as the left arm, in the right leg: the right_2xc_430_2 config
exported asymmetric (right foot 48mm higher than left at zero), so the right leg
was not a mirror of the (correct) left leg. Fixed at model level by mirroring the
left leg onto the right (scripts/mirror_limb.py, generalized from the arm fix).

- Right leg rebuilt as Y-mirror of left (poses/axes/inertials + mirrored meshes).
- Keyframe: both legs use same joint values (mirror convention); ankle solved for
  flat feet (pitch -0.2914, roll -0.0403); base z=0.3052 so feet sit on ground.
- Verified: feet symmetric + flat (0.0deg) + on ground (z=0.002), knee articulation
  mirrors, mass 3.4522 kg, all 6 variants load, physics stable. URDF regenerated.

Co-Authored-By: Claude Opus 4.8 <noreply@anthropic.com>

File: toddlerbot/descriptions/toddlerbot_3_0_2xc/toddlerbot_3_0_2xc.urdf (robot description, URDF)
Before this commit: robot toddlerbot_3_0_2xc, 91 links, 90 joints
Links:
- link right_ankle_pitch_link: geometry collision box size=0.0804121 0.0471454 0.0925345 type=box; visual mesh filename=assets/rightmir_left_ankle_pitch_link_visual.stl scale=1.0 1.0 1.0
- link right_ankle_roll_link: geometry collision box size=0.11 0.042 0.014 type=box; visual mesh filename=assets/rightmir_left_ankle_roll_link_visual.stl scale=1.0 1.0 1.0
- link right_hip_pitch_link: geometry collision box size=0.0409073 0.0409073 0.0465 type=box; visual mesh filename=assets/rightmir_left_hip_pitch_link_visual.stl scale=1.0 1.0 1.0
- link right_hip_roll_link: geometry visual mesh filename=assets/rightmir_left_hip_roll_link_visual.stl scale=1.0 1.0 1.0
- link right_hip_yaw_gear_drive: geometry visual mesh filename=assets/rightmir_left_hip_yaw_gear_drive_visual.stl scale=1.0 1.0 1.0
- link right_hip_yaw_link: geometry collision box size=0.0716062 0.05308 0.0629661 type=box; visual mesh filename=assets/rightmir_left_hip_yaw_link_visual.stl scale=1.0 1.0 1.0
- link right_knee_link: geometry collision box size=0.0394838 0.0515223 0.132305 type=box; visual mesh filename=assets/rightmir_left_knee_link_visual.stl scale=1.0 1.0 1.0
Joints:
- joint right_ankle_pitch: axis -0.221187 -0.975232 0.0 -> -0.221187 0.975232 0.0; limit lower=0.8726646259971649 upper=3.6651914291880923 effort=100 velocity=100 -> lower=0.0 upper=2.879793265790644 effort=100 velocity=100
- joint right_ankle_roll: axis 0.0 0.0 1.0 -> -0.487786 -0.109503 0.866068; origin xyz=-0.00422789 -0.0185236 -0.023 rpy=0.0 0.0 0.0 -> xyz=-0.00698377 -0.0210826 0.0199186 rpy=0.0 0.0 0.0
- joint right_hip_pitch: axis 0.0 -1.0 0.0 -> 0.0 1.0 0.0; limit lower=-1.83259571459404 upper=2.356194490192351 effort=100 velocity=100 -> lower=-2.356194490192344 upper=1.832595714594047 effort=100 velocity=100
- joint right_hip_roll: origin xyz=-0.019 -0.019 -0.024 rpy=0.0 0.0 0.0 -> xyz=0.019 -0.019 -0.024 rpy=0.0 0.0 0.0
- joint right_hip_yaw_drive: origin xyz=-0.0186519 0.00456488 0.0 rpy=0.0 0.0 0.0 -> xyz=-0.0187854 -0.00397992 0.0 rpy=0.0 0.0 0.0
- joint right_hip_yaw_driven: axis 0.0 0.0 -1.0 -> 0.0 0.0 1.0; origin xyz=0.019 0.0 -0.033 rpy=0.0 0.0 0.0 -> xyz=-0.019 0.0 -0.033 rpy=0.0 0.0 0.0
- joint right_knee: axis 0.221187 0.975232 0.0 -> 0.221187 -0.975232 0.0; limit lower=3.552713678800501e-15 upper=2.094395102393199 effort=100 velocity=100 -> lower=-2.0943951023931917 upper=3.552713678800501e-15 effort=100 velocity=100; origin xyz=0.00422789 0.0185236 -0.0445 rpy=0.0 0.0 0.0 -> xyz=-0.00422789 0.0185236 -0.0445 rpy=0.0 0.0 0.0
